File: hardware/roomSensor/HeaterControl.kicad_pcb (KiCad board)
At the start: 2 copper layers, 31.5 x 27.2 mm, 13 parts, among them J1 UART, J2 BTN, J3 OLED, P1 TC2030-CTX, SW1 RESET, U1 DS18B20, U2 BL654, U3 SHT30-DIS-B, U4 Coin Battery

Commit message: Add another schematic, add capacitor and rework 3v3 on laird
Parts:
- added C2: 10uF, Capacitor_Tantalum_SMD:CP_EIA-2012-12_Kemet-R, F.Cu at (119.4, 81.0)
Connections:
- U2 pad 25: +3V3 -> Net-(U2-Pad25)
Routing:
- net +3V3: track 61.9 -> 58.6 mm
- net GND: track 47.0 -> 49.8 mm, vias 32 -> 34
- net /SDA: track 33.2 -> 33.9 mm
Changed lines of the file:
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@@
     (thickness 1.6)
     (drawings 11)
-    (tracks 217)
+    (tracks 224)
     (zones 0)
-    (modules 13)
-    (nets 58)
+    (modules 14)
+    (nets 59)
   )
   (page A4)
@@
   (net 56 "Net-(U2-Pad42)")
   (net 57 "Net-(U2-Pad9)")
+  (net 58 "Net-(U2-Pad25)")
   (net_class Default "This is the default net class."
     (clearance 0.2)
@@
     (add_net "Net-(U2-Pad22)")
     (add_net "Net-(U2-Pad24)")
+    (add_net "Net-(U2-Pad25)")
     (add_net "Net-(U2-Pad27)")
     (add_net "Net-(U2-Pad28)")
@@
     (uvia_dia 0.3)
     (uvia_drill 0.1)
+  )
+  (module Capacitor_Tantalum_SMD:CP_EIA-2012-12_Kemet-R (layer F.Cu)
+    (at 119.38 81.026 270)
+    (descr "Tantalum Capacitor SMD Kemet-R (2012-12 Metric), IPC_7351 nominal, (Body size from: https://www.vishay.com/docs/40182/tmch.pdf), generated with kicad-footprint-generator")
+    (tags "capacitor tantalum")
+    (attr smd)
+    (fp_text reference C2 (at 0 -1.58 270) (layer F.SilkS) hide
+      (effects (font (size 1 1) (thickness 0.15)))
+    )
+    (fp_text value 10uF (at -0.508 -1.524 90) (layer F.Fab)
+      (effects (font (size 0.5 0.5) (thickness 0.08)))
+    )
+    (fp_line (start 1 -0.625) (end -0.6875 -0.625) (layer F.Fab) (width 0.1))
+    (fp_line (start -0.6875 -0.625) (end -1 -0.3125) (layer F.Fab) (width 0.1))
+    (fp_line (start -1 -0.3125) (end -1 0.625) (layer F.Fab) (width 0.1))
+    (fp_line (start -1 0.625) (end 1 0.625) (layer F.Fab) (width 0.1))
+    (fp_line (start 1 0.625) (end 1 -0.625) (layer F.Fab) (width 0.1))
+    (fp_line (start 1 -0.785) (end -1.71 -0.785) (layer F.SilkS) (width 0.12))
+    (fp_line (start -1.71 -0.785) (end -1.71 0.785) (layer F.SilkS) (width 0.12))
+    (fp_line (start -1.71 0.785) (end 1 0.785) (layer F.SilkS) (width 0.12))
+    (fp_line (start -1.7 0.88) (end -1.7 -0.88) (layer F.CrtYd) (width 0.05))
+    (fp_line (start -1.7 -0.88) (end 1.7 -0.88) (layer F.CrtYd) (width 0.05))
+    (fp_line (start 1.7 -0.88) (end 1.7 0.88) (layer F.CrtYd) (width 0.05))
+    (fp_line (start 1.7 0.88) (end -1.7 0.88) (layer F.CrtYd) (width 0.05))
+    (fp_text user %R (at 0 0 270) (layer F.Fab)
+      (effects (font (size 0.5 0.5) (thickness 0.08)))
+    )
+    (pad 1 smd roundrect (at -0.8875 0 270) (size 1.125 1.05) (layers F.Cu F.Paste F.Mask) (roundrect_rratio 0.238095)
+      (net 1 +3V3))
+    (pad 2 smd roundrect (at 0.8875 0 270) (size 1.125 1.05) (layers F.Cu F.Paste F.Mask) (roundrect_rratio 0.238095)
+      (net 3 GND))
+    (model ${KISYS3DMOD}/Capacitor_Tantalum_SMD.3dshapes/CP_EIA-2012-12_Kemet-R.wrl
+      (at (xyz 0 0 0))
+      (scale (xyz 1 1 1))
+      (rotate (xyz 0 0 0))
+    )
   )
   (module Connector_PinHeader_2.54mm:PinHeader_1x02_P2.54mm_Vertical (layer F.Cu)
@@
       (net 14 "Net-(U2-Pad27)"))
     (pad 25 smd rect (at 2.8 9.55) (size 0.5 0.5) (layers F.Cu F.Paste F.Mask)
-      (net 1 +3V3))
+      (net 58 "Net-(U2-Pad25)"))
     (pad 24 smd rect (at 3.6 9.55) (size 0.5 0.5) (layers F.Cu F.Paste F.Mask)
       (net 15 "Net-(U2-Pad24)"))
@@
   (segment (start 130.302 83.566) (end 130.302 80.838) (width 0.4) (layer F.Cu) (net 1))
   (segment (start 130.302 86.106) (end 130.302 83.566) (width 0.4) (layer F.Cu) (net 1))
-  (segment (start 115.676 78.74) (end 117.608 78.74) (width 0.4) (layer F.Cu) (net 1))
-  (segment (start 115.208 78.272) (end 115.676 78.74) (width 0.4) (layer F.Cu) (net 1))
-  (segment (start 115.208 77.622) (end 115.208 78.272) (width 0.4) (layer F.Cu) (net 1))
-  (segment (start 117.608 78.74) (end 117.608 77.622) (width 0.4) (layer F.Cu) (net 1))
-  (segment (start 122.327997 83.715999) (end 130.152001 83.715999) (width 0.4) (layer F.Cu) (net 1))
-  (segment (start 117.608 78.996002) (end 122.327997 83.715999) (width 0.4) (layer F.Cu) (net 1))
-  (segment (start 117.608 78.74) (end 117.608 78.996002) (width 0.4) (layer F.Cu) (net 1))
   (segment (start 113.408 88.392) (end 113.662 88.138) (width 0.4) (layer F.Cu) (net 1))
   (segment (start 106.426 88.392) (end 113.408 88.392) (width 0.4) (layer F.Cu) (net 1))
   (segment (start 113.662 85.09) (end 113.662 82.042) (width 0.4) (layer F.Cu) (net 1))
-  (segment (start 113.662 80.987998) (end 113.662 81.067) (width 0.4) (layer F.Cu) (net 1))
-  (segment (start 115.676 78.973998) (end 113.662 80.987998) (width 0.4) (layer F.Cu) (net 1))
-  (segment (start 113.662 81.067) (end 113.662 82.042) (width 0.4) (layer F.Cu) (net 1))
-  (segment (start 115.676 78.74) (end 115.676 78.973998) (width 0.4) (layer F.Cu) (net 1))
   (segment (start 113.662 88.138) (end 113.662 86.614) (width 0.4) (layer F.Cu) (net 1))
   (segment (start 113.662 86.614) (end 113.662 85.09) (width 0.4) (layer F.Cu) (net 1))
@@
   (segment (start 118.1355 86.614) (end 119.634 88.1125) (width 0.4) (layer F.Cu) (net 1))
   (segment (start 113.662 86.614) (end 118.1355 86.614) (width 0.4) (layer F.Cu) (net 1))
+  (segment (start 128.3295 80.1385) (end 128.966 79.502) (width 0.4) (layer F.Cu) (net 1))
+  (segment (start 119.38 80.1385) (end 128.3295 80.1385) (width 0.4) (layer F.Cu) (net 1))
+  (segment (start 115.208 78.272) (end 115.208 77.622) (width 0.4) (layer F.Cu) (net 1))
+  (segment (start 116.880001 78.272001) (end 115.208 78.272) (width 0.4) (layer F.Cu) (net 1))
+  (segment (start 118.7465 80.1385) (end 116.880001 78.272001) (width 0.4) (layer F.Cu) (net 1))
+  (segment (start 119.38 80.1385) (end 118.7465 80.1385) (width 0.4) (layer F.Cu) (net 1))
+  (segment (start 115.354001 78.418001) (end 115.208 78.272) (width 0.4) (layer F.Cu) (net 1))
+  (segment (start 115.354001 79.124001) (end 115.354001 78.418001) (width 0.4) (layer F.Cu) (net 1))
+  (segment (start 114.35771 80.120292) (end 115.354001 79.124001) (width 0.4) (layer F.Cu) (net 1))
+  (segment (start 114.35771 81.34629) (end 114.35771 80.120292) (width 0.4) (layer F.Cu) (net 1))
+  (segment (start 113.662 82.042) (end 114.35771 81.34629) (width 0.4) (layer F.Cu) (net 1))
   (via (at 109.648448 82.470448) (size 0.8) (drill 0.4) (layers F.Cu B.Cu) (net 2))
   (segment (start 113.608 78.510896) (end 109.648448 82.470448) (width 0.25) (layer F.Cu) (net 2))
@@
   (segment (start 122.174 88.646) (end 122.428 88.9) (width 0.4) (layer F.Cu) (net 3))
   (segment (start 122.174 86.36) (end 122.174 88.646) (width 0.4) (layer F.Cu) (net 3))
+  (via (at 120.904 82.042) (size 0.8) (drill 0.4) (layers F.Cu B.Cu) (net 3))
+  (via (at 119.38 83.058) (size 0.8) (drill 0.4) (layers F.Cu B.Cu) (net 3))
+  (segment (start 119.5085 82.042) (end 119.38 81.9135) (width 0.4) (layer F.Cu) (net 3))
+  (segment (start 120.904 82.042) (end 119.5085 82.042) (width 0.4) (layer F.Cu) (net 3))
+  (segment (start 119.38 81.9135) (end 119.38 83.058) (width 0.4) (layer F.Cu) (net 3))
   (segment (start 126.353571 69.076571) (end 126.746 69.469) (width 0.25) (layer F.Cu) (net 4))
   (segment (start 120.327569 69.076571) (end 126.353571 69.076571) (width 0.25) (layer F.Cu) (net 4))
@@
   (segment (start 129.126999 87.470999) (end 129.452001 87.796001) (width 0.25) (layer F.Cu) (net 8))
   (segment (start 125.179409 87.470999) (end 129.126999 87.470999) (width 0.25) (layer F.Cu) (net 8))
-  (segment (start 119.75041 82.042) (end 125.179409 87.470999) (width 0.25) (layer F.Cu) (net 8))
-  (segment (start 116.462 82.042) (end 119.75041 82.042) (width 0.25) (layer F.Cu) (net 8))
   (via (at 116.078 75.946) (size 0.8) (drill 0.4) (layers F.Cu B.Cu) (net 8))
   (segment (start 113.984 75.946) (end 116.078 75.946) (width 0.25) (layer F.Cu) (net 8))
@@
   (segment (start 116.476 82.028) (end 116.462 82.042) (width 0.25) (layer F.Cu) (net 8))
   (segment (start 116.476 79.54) (end 116.476 82.028) (width 0.25) (layer F.Cu) (net 8))
+  (segment (start 116.462 82.042) (end 116.462 83.188) (width 0.25) (layer F.Cu) (net 8))
+  (segment (start 122.3484 84.63999) (end 125.179409 87.470999) (width 0.25) (layer F.Cu) (net 8))
+  (segment (start 117.91399 84.63999) (end 122.3484 84.63999) (width 0.25) (layer F.Cu) (net 8))
+  (segment (start 116.462 83.188) (end 117.91399 84.63999) (width 0.25) (layer F.Cu) (net 8))
   (segment (start 127.266 88.15) (end 127.762 88.646) (width 0.25) (layer F.Cu) (net 9))
   (segment (start 125.222 88.15) (end 127.266 88.15) (width 0.25) (layer F.Cu) (net 9))
